Commit message: :bug: fixed some bugs

File: description/ros2_control/hoverboard_driver.ros2_control.xacro (robot description, xacro)
@@ -7,5 +7,5 @@
         <param name="wheel_radius">0.0825</param>
         <param name="max_velocity">1.0</param>
-        <param name="device">/dev/serial/by-id/usb-FTDI_Quad_RS232-HS-if01-port0</param>
+        <param name="device">/dev/ttyUSB0</param>
       </hardware>
       <joint name="${prefix}left_wheel_joint">

File: description/urdf/diffbot_description.urdf.xacro (robot description, xacro)
@@ -10,5 +10,5 @@
   <xacro:property name="wheel_mass" value="0.3" /> <!-- arbitrary value for wheel mass -->
   <xacro:property name="wheel_len" value="0.020" />
-  <xacro:property name="wheel_radius" value="0.015" />
+  <xacro:property name="wheel_radius" value="0.08" />
   <xacro:property name="caster_wheel_mass" value="0.1" /> <!-- arbitrary value for caster wheel mass -->
   <xacro:property name="caster_wheel_radius" value="0.015" />
